Commit message: namespace fixed

File: turtlebot3_manipulation/turtlebot3_manipulation_description/urdf/open_manipulator_x.urdf.xacro (robot description, xacro)
@@ -182,9 +182,4 @@
       </inertial>
     </link>
-    <joint name="${prefix}gripper_right_joint_mimic" type="fixed">
-      <parent link="${prefix}link5" />
-      <child link="dummy_mimic_fix" />
-    </joint>
-    <link name="dummy_mimic_fix"/>
     <joint name="${prefix}gripper_right_joint" type="prismatic">
       <parent link="${prefix}link5"/>

File: turtlebot3_simulations/turtlebot3_manipulation_gazebo/gazebo/turtlebot3_waffle_pi.gazebo.xacro (robot description, xacro)
@@ -65,6 +65,6 @@
         <remapping>odom:=odom</remapping>
       </ros>
-      <left_joint>wheel_left_joint</left_joint>
-      <right_joint>wheel_right_joint</right_joint>
+      <left_joint>manipulator/wheel_left_joint</left_joint>
+      <right_joint>manipulator/manipulator/wheel_right_joint</right_joint>
       <wheel_separation>0.287</wheel_separation>
       <wheel_diameter>0.066</wheel_diameter>
@@ -123,6 +123,6 @@
           <horizontal_fov>1.02974</horizontal_fov>
           <image>
-              <width>1920</width>
-              <height>1080</height>
+              <width>640</width>
+              <height>480</height>
               <format>R8G8B8</format>
           </image>
@@ -174,5 +174,7 @@
       filename="libgazebo_ros_camera.so">
       <ros>
-        <!-- <namespace>/manipulator</namespace> -->
+        <namespace>manipulator</namespace>
+        <remapping>image_raw:=camera/depth/rgb_raw</remapping>
+        <remapping>camera_info:=camera/depth/rgb_info</remapping>
         <remapping>camera/depth/image_raw:=camera/depth/image_raw</remapping>
         <remapping>camera/depth/camera_info:=camera/depth/camera_info</remapping>

File: turtlebot3_simulations/turtlebot3_manipulation_gazebo/ros2_control/turtlebot3_manipulation_system.ros2_control.xacro (robot description, xacro)
@@ -92,5 +92,5 @@
         </state_interface>
       </sensor>
-      <joint name="joint1">
+      <joint name="${prefix}joint1">
         <command_interface name="position">
           <param name="min">${-pi*0.9}</param>
@@ -104,5 +104,5 @@
         </state_interface>
       </joint>
-      <joint name="joint2">
+      <joint name="${prefix}joint2">
         <command_interface name="position">
           <param name="min">${-pi*0.57}</param>
@@ -116,5 +116,5 @@
         </state_interface>
       </joint>
-      <joint name="joint3">
+      <joint name="${prefix}joint3">
         <command_interface name="position">
           <param name="min">${-pi*0.3}</param>
@@ -128,5 +128,5 @@
         </state_interface>
       </joint>
-      <joint name="joint4">
+      <joint name="${prefix}joint4">
         <command_interface name="position">
           <param name="min">${-pi*0.57}</param>
@@ -140,5 +140,5 @@
         </state_interface>
       </joint>
-      <joint name="gripper_left_joint">
+      <joint name="${prefix}gripper_left_joint">
         <command_interface name="position">
           <param name="min">-0.010</param>
@@ -152,6 +152,6 @@
         </state_interface>
       </joint>
-      <joint name="gripper_right_joint">
-        <param name="mimic">gripper_left_joint</param>
+      <joint name="${prefix}gripper_right_joint">
+        <param name="mimic">${prefix}gripper_left_joint</param>
         <param name="multiplier">1</param>
         <command_interface name="position">

File: turtlebot3_simulations/turtlebot3_manipulation_gazebo/urdf/open_manipulator_x.urdf.xacro (robot description, xacro)
@@ -32,5 +32,5 @@
       </inertial>
     </link>
-    <joint name="joint1" type="revolute">
+    <joint name="${prefix}joint1" type="revolute">
       <parent link="${prefix}link1"/>
       <child link="${prefix}link2"/>
@@ -62,5 +62,5 @@
       </inertial>
     </link>
-    <joint name="joint2" type="revolute">
+    <joint name="${prefix}joint2" type="revolute">
       <parent link="${prefix}link2"/>
       <child link="${prefix}link3"/>
@@ -92,5 +92,5 @@
       </inertial>
     </link>
-    <joint name="joint3" type="revolute">
+    <joint name="${prefix}joint3" type="revolute">
       <parent link="${prefix}link3"/>
       <child link="${prefix}link4"/>
@@ -122,5 +122,5 @@
       </inertial>
     </link>
-    <joint name="joint4" type="revolute">
+    <joint name="${prefix}joint4" type="revolute">
       <parent link="${prefix}link4"/>
       <child link="${prefix}link5"/>
@@ -152,5 +152,5 @@
       </inertial>
     </link>
-    <joint name="gripper_left_joint" type="prismatic">
+    <joint name="${prefix}gripper_left_joint" type="prismatic">
       <parent link="${prefix}link5"/>
       <child link="${prefix}gripper_left_link"/>
@@ -182,10 +182,5 @@
       </inertial>
     </link>
-    <joint name="gripper_right_joint_mimic" type="fixed">
-      <parent link="${prefix}link5" />
-      <child link="dummy_mimic_fix" />
-    </joint>
-    <link name="dummy_mimic_fix"/>
-    <joint name="gripper_right_joint" type="prismatic">
+    <joint name="${prefix}gripper_right_joint" type="prismatic">
       <parent link="${prefix}link5"/>
       <child link="${prefix}gripper_right_link"/>
@@ -218,5 +213,5 @@
       </inertial>
     </link>
-    <joint name="end_effector_joint" type="fixed">
+    <joint name="${prefix}end_effector_joint" type="fixed">
       <parent link="${prefix}link5"/>
       <child link="${prefix}end_effector_link"/>
